File: 3in1_ELRS_ESC.kicad_pcb (KiCad board)
At the start: 2 copper layers, 35 x 35 mm, 106 parts, among them J2 XT30PW-M, P1 SM08B-SRSS-TB(LF)(SN), Q1 SP40N03GNJ, Q10 SP40N03GNJ, Q11 SP40N03GNJ, Q12 SP40N03GNJ, Q2 SP40N03GNJ, Q3 SP40N03GNJ, Q4 SP40N03GNJ, Q5 SP40N03GNJ, Q6 SP40N03GNJ, Q7 SP40N03GNJ, Q8 SP40N03GNJ, Q9 SP40N03GNJ, U1 AT32F421G8U7, U2 AT32F421G8U7, U3 NSG2065Q_C53463328, U4 NSG2065Q_C53463328, U5 LMR51420YDDCR, U6 TLV76733DRVR, U7 INA186A3IDCKR

Commit message: Routing Trouble
Parts:
- removed M1, M2: ~, TestPoint:TestPoint_THTPad_2.5x2.5mm_Drill1.2mm
- C10, C11, C12, C13, C14, C15, C16, C17, C18, C19, C20, C21, C22, C23, C24, C25, C26, C27, C28, C29, C30, C31, C9, D1, D2, D3, D4, D5, D6, D7, R15, R16, R19, R20, R23, R24, R25, R26, R27, R28, R29, R30, R33, R34, R35, U5, U6, U7: moved to B.Cu
- L1: footprint lcsc_footprints:C1331018_IND-SMD_L12_5-W12_5_B82477P4XX -> lcsc_footprints:C2879693_IND-SMD_L4_5-W4_0; moved to B.Cu
- R36: value RF - 10kΩ -> (none); moved to B.Cu
- moved C22 182.1 mm to (81.6, 107.2), turned to 180 degrees
- moved C27 181.7 mm to (81.6, 109.3), turned to 180 degrees
- moved C28 175.2 mm to (92.6, 106.8), turned to 90 degrees
- moved C21 173.7 mm to (93.8, 110.5), turned to 180 degrees
- moved R33 173.4 mm to (81.2, 103.1), turned to -90 degrees
- moved U5 165.4 mm to (94.8, 106.8)
- moved R34 159.0 mm to (98.1, 108.8), turned to -90 degrees
- moved L1 156.7 mm to (95.8, 101.7), turned to 90 degrees
- moved U7 128.6 mm to (76.6, 103.5), turned to -90 degrees
- moved D7 125.3 mm to (83.5, 116.1)
- moved C31 124.8 mm to (84.6, 99.3), turned to -90 degrees
- moved R35 123.3 mm to (71.7, 111.5), turned to 180 degrees
- moved R36 120.8 mm to (81.1, 99.3), turned to 90 degrees
- moved C10 104.3 mm to (71.7, 101.2), turned to 90 degrees
- moved C19 97.3 mm to (77.9, 112.0)
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Connections:
- C19 pad 1: +BATT -> (no net)
- C20 pad 1: +BATT -> (no net)
- C23 pad 1: +BATT -> (no net)
- C24 pad 1: +BATT -> (no net)
- C25 pad 1: +BATT -> (no net)
- C26 pad 1: +BATT -> (no net)
- Q1 pad 8: +BATT -> (no net)
- Q2 pad 8: +BATT -> (no net)
- Q3 pad 8: +BATT -> (no net)
- Q4 pad 8: +BATT -> (no net)
- Q5 pad 8: +BATT -> (no net)
- Q6 pad 8: +BATT -> (no net)
- U3 pad 4: +BATT -> (no net)
- U4 pad 4: +BATT -> (no net)
- U7 pad 4: +BATT -> (no net)
Routing:
- net /ESC 1/FBC: track 0.00 -> 36.3 mm, vias 0 -> 2
- net /ESC 1/GHA_2: track 0.00 -> 32.1 mm
- net /ESC 1/VB1: track 0.00 -> 25.6 mm
- net /ESC 1/FBB: track 0.00 -> 24.1 mm, vias 0 -> 2
- net /ESC 1/GHB_2: track 0.00 -> 23.4 mm
- net /ESC 1/GLC_2: track 0.00 -> 20.1 mm, vias 0 -> 2
- net /ESC 1/CH: track 0.00 -> 13.8 mm, vias 0 -> 2
- net /ESC 1/GLA_2: track 0.00 -> 13.3 mm, vias 0 -> 2
- net /ESC 1/BH: track 0.00 -> 12.6 mm, vias 0 -> 2
- net /ESC 1/AH: track 0.00 -> 12.5 mm, vias 0 -> 2
- net /ESC 1/FBA: track 0.00 -> 11.5 mm, vias 0 -> 2
- net /ESC 1/CL: track 0.00 -> 6.98 mm, vias 0 -> 2
- net /ESC 1/GHA_1: track 0.00 -> 6.89 mm
- net /ESC 1/GHC_1: track 0.00 -> 6.71 mm
- net /ESC 1/GLB_1: track 0.00 -> 6.03 mm
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- added copper zone on In2.Cu, net +BATT
- added copper zone on In3.Cu, net GND
Other:
- board size 35 x 35 mm -> 40 x 35 mm
- copper layers 2 -> 6
