File: 3in1_ELRS_ESC.kicad_sch (KiCad schematic)
At the start: 32 parts, among them J2 XT30PW-M, P1 SM08B-SRSS-TB(LF)(SN), U5 LMR51420YDDCR, U6 TLV76733DRVR, U7 INA186A3IDCKR

Commit message: Routing Trouble
Parts:
- L1: footprint lcsc_footprints:C1331018_IND-SMD_L12_5-W12_5_B82477P4XX -> lcsc_footprints:C2879693_IND-SMD_L4_5-W4_0; symbol lcsc_imported:SRR1260-4R7Y -> lcsc_imported:CY43-4_7UH; LCSC C1331018 -> C2879693; Manufacturer BOURNS -> SHOU HAN(首韩)
Changed lines of the file:
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@@
 	)
 	(symbol
-		(lib_id "lcsc_imported:SRR1260-4R7Y")
+		(lib_id "lcsc_imported:CY43-4_7UH")
 		(at 245.11 25.4 0)
 		(unit 1)
@@
 			)
 		)
-		(property "Footprint" "lcsc_footprints:C1331018_IND-SMD_L12_5-W12_5_B82477P4XX"
+		(property "Footprint" "lcsc_footprints:C2879693_IND-SMD_L4_5-W4_0"
 			(at 245.11 35.56 0)
 			(hide yes)
@@
 			)
 		)
-		(property "Datasheet" "https://wmsc.lcsc.com/wmsc/upload/file/pdf/v2/lcsc/2304140030_BOURNS-SRR1260-4R7Y_C1331018.pdf"
+		(property "Datasheet" "https://wmsc.lcsc.com/wmsc/upload/file/pdf/v2/lcsc/2108150430_SHOU-HAN-CY43-4-7UH_C2879693.pdf"
 			(at 242.824 25.273 0)
 			(hide yes)
@@
 			)
 		)
-		(property "Description" "SRR1260-4R7Y"
+		(property "Description" "CY43-4.7UH"
 			(at 245.11 25.4 0)
 			(hide yes)
@@
 			)
 		)
-		(property "LCSC" "C1331018"
+		(property "LCSC" "C2879693"
 			(at 245.11 25.4 0)
 			(hide yes)
@@
 			)
 		)
-		(property "Manufacturer" "BOURNS"
+		(property "Manufacturer" "SHOU HAN(首韩)"
 			(at 245.11 25.4 0)
 			(hide yes)
